File: _Vanguard_V2/Vanguard New_1/Vanguard New_1.kicad_sch (KiCad schematic)
At the start: 4 parts, among them J1 USB_B_Micro, J2 Conn_01x03_Pin, U1 ATSAMD11D14A-M

Commit message: small schematic update
Parts:
- added J3: Screw_Terminal_01x02, symbol Connector:Screw_Terminal_01x02
- added Q1: IRLB8721PBF, Package_TO_SOT_THT:TO-220-3_Vertical, symbol Transistor_FET:IRLB8721PBF
- added U2: BNO055, Package_LGA:LGA-28_5.2x3.8mm_P0.5mm, symbol Sensor_Motion:BNO055
- added U3: ATSAMD21G18A-A, Package_QFP:TQFP-48_7x7mm_P0.5mm, symbol MCU_Microchip_SAMD:ATSAMD21G18A-A
- added U4: BMP280, Package_LGA:Bosch_LGA-8_2x2.5mm_P0.65mm_ClockwisePinNumbering, symbol Sensor_Pressure:BMP280
Connections:
- new net: U3.18 (GND), U3.35 (GND), U3.42 (GND)
- new net: U2.15 (GNDIO), U2.16 (GNDIO), U2.25 (GNDIO)
