File: Vanguard/Vanguard_new/Vanguard_new.kicad_pcb (KiCad board)
At the start: 4 copper layers, 628.1 x 251 mm, 70 parts, among them J1 USB_C, J2 Conn_02x03_Pin, J3 Micro_SD_Card_Det1, J4 STARBOARD_SERVO, J5 PORTSIDE_SERVO, Q1 BSS138, Q2 BSS138, Q3 BSS138, Q4 BSS138, U1 ATSAMD11D14A-M, U2 ATmega4809-A, U3 AT25DF641A-SH-T, U4 AP2112K-3.3, U5 MPM3610AGQV-P, U6 BNO086, U7 TXB0104D, U8 TPS61092, Y1 32.768kHz

Commit message: just in case push
Parts:
- moved R15 38.0 mm to (207.7, 36.8)
- moved R16 38.0 mm to (207.7, 38.8)
- moved R17 38.0 mm to (207.7, 40.8)
- moved C5 31.7 mm to (196.7, 28.3)
- moved C6 31.7 mm to (196.7, 34.1)
- moved D5 31.7 mm to (223.4, 34.9)
- moved D6 22.5 mm to (200.0, 36.5)
Changed lines of the file:
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@@
 	(footprint "Resistor_SMD:R_0402_1005Metric"
 		(layer "F.Cu")
-		(at 241.72 21.83)
+		(at 207.69 38.77)
 		(descr "Resistor SMD 0402 (1005 Metric), square (rectangular) end terminal, IPC_7351 nominal, (Body size source: IPC-SM-782 page 72, https://www.pcb-3d.com/wordpress/wp-content/uploads/ipc-sm-782a_amendment_1_and_2.pdf), generated with kicad-footprint-generator")
 		(tags "resistor")
@@
 		)
 		(fp_text user "${REFERENCE}"
-			(at 0 2.54 360)
+			(at 0 2.54 0)
 			(layer "F.Fab")
 			(effects
@@
 	(footprint "LED_SMD:LED_0201_0603Metric"
 		(layer "F.Cu")
-		(at 248.99 53.62)
+		(at 223.43 34.86)
 		(descr "LED SMD 0201 (0603 Metric), square (rectangular) end terminal, IPC_7351 nominal, (Body size source: https://www.vishay.com/docs/20052/crcw0201e3.pdf), generated with kicad-footprint-generator")
 		(tags "LED")
@@
 		(tags "USB Type-C Plug Edge Mount")
 		(property "Reference" "J1"
-			(at 3.24 -70.5 360)
+			(at 3.24 -70.5 0)
 			(layer "F.SilkS")
 			(effects
@@
 		)
 		(property "Value" "USB_C"
-			(at 0 -1.96 360)
+			(at 0 -1.96 0)
 			(layer "F.Fab")
 			(effects
@@
 		)
 		(fp_text user "PCB Edge"
-			(at 0 -0.96 360)
+			(at 0 -0.96 0)
 			(layer "Dwgs.User")
 			(effects
@@
 		)
 		(fp_text user "${REFERENCE}"
-			(at 0 2.04 360)
+			(at 0 2.04 0)
 			(layer "F.Fab")
 			(effects
@@
 		(tags "capacitor")
 		(property "Reference" "C7"
-			(at 0 -1.05 360)
+			(at 0 -1.05 0)
 			(layer "F.SilkS")
 			(effects
@@
 		)
 		(property "Value" "0.1uF"
-			(at 0 1.05 360)
+			(at 0 1.05 0)
 			(layer "F.Fab")
 			(effects
@@
 		)
 		(fp_text user "${REFERENCE}"
-			(at 0 -0.68 360)
+			(at 0 -0.68 0)
 			(layer "F.Fab")
 			(effects
@@
 		(tags "resistor")
 		(property "Reference" "R23"
-			(at 0 -1.17 360)
+			(at 0 -1.17 0)
 			(layer "F.SilkS")
 			(effects
@@
 		)
 		(property "Value" "10k"
-			(at 0 1.17 360)
+			(at 0 1.17 0)
 			(layer "F.Fab")
 			(effects
@@
 		)
 		(fp_text user "${REFERENCE}"
-			(at 0 0 360)
+			(at 0 0 0)
 			(layer "F.Fab")
 			(effects
@@
 		(tags "resistor")
 		(property "Reference" "R26"
-			(at 0 -1.17 360)
+			(at 0 -1.17 0)
 			(layer "F.SilkS")
 			(effects
@@
 		)
 		(property "Value" "220"
-			(at 0 1.17 360)
+			(at 0 1.17 0)
 			(layer "F.Fab")
 			(effects
@@
 		)
 		(fp_text user "${REFERENCE}"
-			(at 0 0 360)
+			(at 0 0 0)
 			(layer "F.Fab")
 			(effects
@@
 		(tags "resistor")
 		(property "Reference" "R29"
-			(at 0 -1.17 360)
+			(at 0 -1.17 0)
 			(layer "F.SilkS")
 			(effects
@@
 		)
 		(property "Value" "220"
-			(at 0 1.17 360)
+			(at 0 1.17 0)
 			(layer "F.Fab")
 			(effects
@@
 		)
 		(fp_text user "${REFERENCE}"
-			(at 0 0 360)
+			(at 0 0 0)
 			(layer "F.Fab")
 			(effects
@@
 		(tags "capacitor")
 		(property "Reference" "C2"
-			(at 28.55 -0.18 360)
+			(at 28.55 -0.18 0)
 			(layer "F.SilkS")
 			(effects
@@
 		)
 		(property "Value" "22pF"
-			(at 28.55 1.92 360)
+			(at 28.55 1.92 0)
 			(layer "F.Fab")
 			(effects
@@
 		)
 		(fp_text user "${REFERENCE}"
-			(at 0 -0.68 360)
+			(at 0 -0.68 0)
 			(layer "F.Fab")
 			(effects
@@
 	(footprint "Resistor_SMD:R_0402_1005Metric"
 		(layer "F.Cu")
-		(at 241.72 23.82)
+		(at 207.69 40.76)
 		(descr "Resistor SMD 0402 (1005 Metric), square (rectangular) end terminal, IPC_7351 nominal, (Body size source: IPC-SM-782 page 72, https://www.pcb-3d.com/wordpress/wp-content/uploads/ipc-sm-782a_amendment_1_and_2.pdf), generated with kicad-footprint-generator")
 		(tags "resistor")
@@
 		(tags "capacitor")
 		(property "Reference" "C3"
-			(at 28.55 -0.18 360)
+			(at 28.55 -0.18 0)
 			(layer "F.SilkS")
 			(effects
@@
 		)
 		(property "Value" "22pF"
-			(at 28.55 1.92 360)
+			(at 28.55 1.92 0)
 			(layer "F.Fab")
 			(effects
@@
 		)
 		(fp_text user "${REFERENCE}"
-			(at 0 -0.68 360)
+			(at 0 -0.68 0)
 			(layer "F.Fab")
 			(effects
@@
 		(tags "LED ROHM SMLVN6")
 		(property "Reference" "PORTSIDE_RGB1"
-			(at 0 -2.65 360)
+			(at 0 -2.65 0)
 			(layer "F.SilkS")
 			(effects
@@
 		)
 		(property "Value" "SMLVN6RGB"
-			(at 0 2.65 360)
+			(at 0 2.65 0)
 			(layer "F.Fab")
 			(effects
@@
 		)
 		(fp_text user "${REFERENCE}"
-			(at 0 0 360)
+			(at 0 0 0)
 			(layer "F.Fab")
 			(effects
@@
 		(tags "resistor")
 		(property "Reference" "R25"
-			(at 0 -1.17 360)
+			(at 0 -1.17 0)
 			(layer "F.SilkS")
 			(effects
@@
 		)
 		(property "Value" "220"
-			(at 0 1.17 360)
+			(at 0 1.17 0)
 			(layer "F.Fab")
 			(effects
@@
 		)
 		(fp_text user "${REFERENCE}"
-			(at 0 0 360)
+			(at 0 0 0)
 			(layer "F.Fab")
 			(effects
@@
 	(footprint "Diode_SMD:Nexperia_CFP3_SOD-123W"
 		(layer "F.Cu")
-		(at 183.82 52.17 90)
+		(at 199.96 36.46 90)
 		(descr "Nexperia CFP3 (SOD-123W), https://assets.nexperia.com/documents/outline-drawing/SOD123W.pdf")
 		(tags "CFP3 SOD-123W")
@@
 		(tags "resistor")
 		(property "Reference" "R27"
-			(at 0 -1.17 360)
+			(at 0 -1.17 0)
 			(layer "F.SilkS")
 			(effects
@@
 		)
 		(property "Value" "220"
-			(at 0 1.17 360)
+			(at 0 1.17 0)
 			(layer "F.Fab")
 			(effects
@@
 		)
 		(fp_text user "${REFERENCE}"
-			(at 0 0 360)
+			(at 0 0 0)
 			(layer "F.Fab")
 			(effects
@@
 		(tags "resistor")
 		(property "Reference" "R28"
-			(at 0 -1.17 360)
+			(at 0 -1.17 0)
 			(layer "F.SilkS")
 			(effects
@@
 		)
 		(property "Value" "220"
-			(at 0 1.17 360)
+			(at 0 1.17 0)
 			(layer "F.Fab")
 			(effects
@@
 		)
 		(fp_text user "${REFERENCE}"
-			(at 0 0 360)
+			(at 0 0 0)
 			(layer "F.Fab")
 			(effects
@@
 		(tags "resistor")
 		(property "Reference" "R30"
-			(at 0 -1.17 360)
+			(at 0 -1.17 0)
 			(layer "F.SilkS")
 			(effects
@@
 		)
 		(property "Value" "220"
-			(at 0 1.17 360)
+			(at 0 1.17 0)
 			(layer "F.Fab")
 			(effects
@@
 		)
 		(fp_text user "${REFERENCE}"
-			(at 0 0 360)
+			(at 0 0 0)
 			(layer "F.Fab")
 			(effects
@@
 		(tags "net tie solder jumper bridged")
 		(property "Reference" "ADR1"
-			(at 0 -1.8 360)
+			(at 0 -1.8 0)
 			(layer "F.SilkS")
 			(effects
@@
 		)
 		(property "Value" "~"
-			(at 0 1.9 360)
+			(at 0 1.9 0)
 			(layer "F.Fab")
 			(effects
@@
 		(tags "LED ROHM SMLVN6")
 		(property "Reference" "STARBOARD_RGB1"
-			(at 0 -2.65 360)
+			(at 0 -2.65 0)
 			(layer "F.SilkS")
 			(effects
@@
 		)
 		(property "Value" "SMLVN6RGB"
-			(at 0 2.65 360)
+			(at 0 2.65 0)
 			(layer "F.Fab")
 			(effects
@@
 		)
 		(fp_text user "${REFERENCE}"
-			(at 0 0 360)
+			(at 0 0 0)
 			(layer "F.Fab")
 			(effects
@@
 		(tags "buzzer")
 		(property "Reference" "BZ1"
-			(at 2.5 -7.17 360)
+			(at 2.5 -7.17 0)
 			(layer "F.SilkS")
 			(effects
@@
 		)
 		(property "Value" "Buzzer"
-			(at 2.5 7.31 360)
+			(at 2.5 7.31 0)
 			(layer "F.Fab")
 			(effects
@@
 		)
 		(fp_text user "${REFERENCE}"
-			(at 3.736569 64.75 360)
+			(at 3.736569 64.75 0)
 			(layer "F.Fab")
 			(effects
@@
 		)
 		(fp_text user "${REFERENCE}"
-			(at 0 0 360)
+			(at 0 0 0)
 			(layer "F.Fab")
 			(effects
@@
 		(tags "CONN DEV")
 		(property "Reference" "TP2"
-			(at 9.1 -78.62 360)
+			(at 9.1 -78.62 0)
 			(layer "F.SilkS")
 			(effects
@@
 		)
 		(property "Value" "TestPoint"
-			(at 9.1 -73.12 360)
+			(at 9.1 -73.12 0)
 			(layer "F.Fab")
 			(effects
@@
 		)
 		(fp_text user "${REFERENCE}"
-			(at 2.54 0 360)
+			(at 2.54 0 0)
 			(layer "F.Fab")
 			(effects
@@
 	(footprint "Resistor_SMD:R_0402_1005Metric"
 		(layer "F.Cu")
-		(at 241.72 19.84)
+		(at 207.69 36.78)
 		(descr "Resistor SMD 0402 (1005 Metric), square (rectangular) end terminal, IPC_7351 nominal, (Body size source: IPC-SM-782 page 72, https://www.pcb-3d.com/wordpress/wp-content/uploads/ipc-sm-782a_amendment_1_and_2.pdf), generated with kicad-footprint-generator")
 		(tags "resistor")
@@
 		(tags "CONN DEV")
 		(property "Reference" "TP1"
-			(at 2.54 -2.5 360)
+			(at 2.54 -2.5 0)
 			(layer "F.SilkS")
 			(effects
@@
 		)
 		(property "Value" "TestPoint"
-			(at 2.54 3 360)
+			(at 2.54 3 0)
 			(layer "F.Fab")
 			(effects
@@
 		)
 		(fp_text user "${REFERENCE}"
-			(at 2.54 0 360)
+			(at 2.54 0 0)
 			(layer "F.Fab")
 			(effects
@@
 		(tags "SOT TO_SOT_SMD")
 		(property "Reference" "Q4"
-			(at 0 -2.4 360)
+			(at 0 -2.4 0)
 			(layer "F.SilkS")
 			(effects
@@
 		)
 		(property "Value" "BSS138"
-			(at 0 2.4 360)
+			(at 0 2.4 0)
 			(layer "F.Fab")
 			(effects
@@
 		)
 		(fp_text user "${REFERENCE}"
-			(at 0 0 360)
+			(at 0 0 0)
 			(layer "F.Fab")
 			(effects
@@
 	(footprint "Capacitor_SMD:C_0201_0603Metric"
 		(layer "F.Cu")
-		(at 222.285 47.04)
+		(at 196.725 28.28)
 		(descr "Capacitor SMD 0201 (0603 Metric), square (rectangular) end terminal, IPC_7351 nominal, (Body size source: https://www.vishay.com/docs/20052/crcw0201e3.pdf), generated with kicad-footprint-generator")
 		(tags "capacitor")
@@
 		(tags "SOIC SO")
 		(property "Reference" "U7"
-			(at 24.605 -68.09 360)
+			(at 24.605 -68.09 0)
 			(layer "F.SilkS")
 			(effects
@@
 		)
 		(property "Value" "TXB0104D"
-			(at 0 5.28 360)
+			(at 0 5.28 0)
 			(layer "F.Fab")
 			(effects
@@
 		)
 		(fp_text user "${REFERENCE}"
-			(at 5.74 21.9525 360)
+			(at 5.74 21.9525 0)
 			(layer "F.Fab")
 			(effects
@@
 	(footprint "Capacitor_SMD:C_0201_0603Metric"
 		(layer "F.Cu")
-		(at 222.285 52.89)
+		(at 196.725 34.13)
 		(descr "Capacitor SMD 0201 (0603 Metric), square (rectangular) end terminal, IPC_7351 nominal, (Body size source: https://www.vishay.com/docs/20052/crcw0201e3.pdf), generated with kicad-footprint-generator")
 		(tags "capacitor")

Commit message: power stabilization done
Parts:
- moved C6 176.8 mm to (373.2, 23.5), turned to 180 degrees
- moved C5 172.8 mm to (369.5, 25.7), turned to 90 degrees
- moved R17 169.1 mm to (376.0, 25.0)
- moved D6 163.2 mm to (363.0, 30.0), turned to 180 degrees
- moved U4 162.9 mm to (373.0, 26.0)
- moved R16 160.9 mm to (368.0, 25.0)
- moved R15 160.7 mm to (368.0, 26.0), turned to 180 degrees
- moved U5 159.1 mm to (363.4, 26.4), turned to 90 degrees
- moved R14 156.6 mm to (359.5, 27.0)
- moved C4 155.4 mm to (359.5, 25.0)
- moved D5 152.9 mm to (376.0, 26.0)
- moved L1 30.2 mm to (268.5, 130.0), turned to 135 degrees
- moved C8 18.7 mm to (272.0, 128.0), turned to -135 degrees
- moved C9 13.2 mm to (266.0, 128.0), turned to -45 degrees
- moved C10 13.2 mm to (265.5, 128.5), turned to -45 degrees
Routing:
- net GND: track 12.0 -> 31.0 mm, vias 6 -> 13
- net VBUS_out: track 0.00 -> 15.0 mm
- net Net-(U5-FB): track 0.00 -> 9.03 mm, vias 0 -> 2
- net Net-(U4-EN): track 0.00 -> 6.51 mm
- net RST: track 35.7 -> 38.9 mm
- net +5V: track 0.00 -> 2.97 mm
- net Net-(L1-Pad2): track 0.00 -> 1.99 mm
- net Net-(D5-A): track 0.00 -> 1.08 mm
- net Net-(U5-VIN): track 3.42 -> 2.85 mm
- added copper zone on B.Cu, net GND
- removed copper zone on B.Cu, net (none)
- removed copper zone on F.Cu, net (none)
- removed copper zone on In1.Cu, net GND
- removed copper zone on In2.Cu, net GND
Other:
- board size 628.1 x 251 mm -> 683.3 x 251 mm
