File: Vanguard/Vanguard_new/Vanguard_new.kicad_pcb (KiCad board)
At the start: 4 copper layers, 46.2 x 50.9 mm, 74 parts, among them J1 USB_C, J2 Conn_02x03_Pin, J3 Micro_SD_Card_Det1, J4 STARBOARD_SERVO, J5 PORTSIDE_SERVO, J6 Conn_01x02_Pin, Q1 BSS138, Q2 BSS138, Q3 BSS138, Q4 BSS138, U1 ATSAMD11D14A-M, U2 ATmega4809-A, U3 AT25DF641A-SH-T, U4 AP2112K-3.3, U5 MPM3610AGQV-P, U6 BNO086, U7 TXB0104D, U8 TPS61092, Y1 32.768kHz

Commit message: fixed many errors
Parts:
- U8: footprint Package_DFN_QFN:Texas_RSA_VQFN-16-1EP_4x4mm_P0.65mm_EP2.7x2.7mm_ThermalVias -> Package_DFN_QFN:DFN-10-1EP_3x3mm_P0.5mm_EP1.65x2.38mm_ThermalVias
Routing:
- net Net-(U5-FB): track 1.15 -> 10.8 mm, vias 0 -> 2
- net GND: track 80.8 -> 88.2 mm, vias 27 -> 28
- net Net-(L1-Pad2): track 1.99 -> 2.88 mm
