File: Vanguard/Vanguard_dev.kicad_sch (KiCad schematic)
At the start: 96 parts, among them J1 USB_C, J2 Conn_02x03_Pin, J3 Micro_SD_Card_Det1, J4 STARBOARD_SERVO, J5 PORTSIDE_SERVO, J6 Conn_01x02_Pin, Q1 BSS138, Q2 BSS138, Q3 BSS138, Q4 BSS138, U1 ATSAMD11D14A-M, U2 ATmega4809-A, U3 AT25DF641A-SH-T, U4 AP2112K-3.3, U5 MPM3610AGQV-P, U6 BNO086, U7 TXB0104D, U8 TPS61092, Y1 32.768kHz

Commit message: dev_file_changes( same as the v2 one)
Parts:
- removed J1: USB_C, Connector_USB:USB_C_Plug_Molex_105444, symbol Connector:USB_C_Plug_USB2.0
- removed TP10, TP11, TP12, TP15, TP16, TP17, TP18, TP19, TP20, TP21, TP22, TP23, TP24, TP25, TP26, TP27, TP28, TP3, TP4, TP5, TP6, TP7, TP8, TP9: TestPoint, symbol Connector:TestPoint
- added J7: USB_B_Micro, Connector_USB:USB_Micro-B_Wuerth_614105150721_Vertical_CircularHoles, symbol Connector:USB_B_Micro
Connections:
- net GND: now also J7.5 (GND), J7.6 (Shield)
- net VCC: now also C1.1, D1.1 (GND), R1.1, J7.1 (VBUS)
- net at D1.2 (I/O1), TP1.1, U1.22 (PA25): now also J7.2 (D-)
- net at D1.3 (I/O2), TP2.1, U1.21 (PA24): now also J7.3 (D+)

Commit message: Added tespoints
Parts:
- added TP10, TP11, TP12, TP13, TP14, TP15, TP16, TP19, TP20, TP21, TP22, TP23, TP24, TP25, TP26, TP27, TP3, TP4, TP5, TP6, TP7, TP8, TP9: TestPoint, symbol Connector:TestPoint
Connections:
- net +3.3V: now also TP14.1
- net D4: now also TP20.1
- net D5: now also TP19.1
- net D6: now also TP21.1
- net D7: now also TP22.1
- net PORT_BLUE: now also TP8.1
- net PORT_GREEN: now also TP10.1
- net PORT_RED: now also TP9.1
- net SCL: now also TP15.1
- net SDA: now also TP16.1
- net at C2.1, U6.26 (XOUT32/CLKSEL1), Y1.1: now also TP13.1
- net at C3.1, U6.27 (XIN32), Y1.2: now also TP12.1

Commit message: Revert "Added testpoints"
This reverts commit b260b8998230daf1f71bd3849bf22839f1098abd.
Parts:
- removed TP10, TP11, TP12, TP13, TP14, TP15, TP16, TP19, TP20, TP21, TP22, TP23, TP24, TP25, TP26, TP27, TP3, TP4, TP5, TP6, TP7, TP8, TP9: TestPoint, symbol Connector:TestPoint

Commit message: Added_testpoints
Parts:
- added TP10, TP11, TP12, TP13, TP14, TP15, TP16, TP17, TP18, TP19, TP20, TP21, TP22, TP23, TP24, TP25, TP26, TP27, TP28, TP29, TP3, TP30, TP31, TP32, TP33, TP4, TP5, TP6, TP7, TP8, TP9: TestPoint, symbol Connector:TestPoint
Connections:
- net +3.3V: now also TP23.1, TP27.1, TP30.1, TP32.1
- net PORT_BLUE: now also TP8.1
- net PORT_GREEN: now also TP10.1
- net PORT_RED: now also TP9.1
- net RX0: now also TP28.1
- net SCL: now also TP21.1
- net SDA: now also TP20.1
- net STAR_BLUE: now also TP5.1
- net STAR_GREEN: now also TP7.1
- net STAR_RED: now also TP6.1
- net TX0: now also TP29.1
- net VCC: now also TP31.1
- net at C2.1, U6.26 (XOUT32/CLKSEL1), Y1.1: now also TP25.1
- net at C3.1, U6.27 (XIN32), Y1.2: now also TP24.1
- net at C5.1, R15.1, U4.1 (VIN)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: now also TP26.1
