File: Vanguard/Vanguard 2.3/Vanguard_new.kicad_pcb (KiCad board)
At the start: 4 copper layers, 50 x 41.2 mm, 78 parts, among them J1 USB_C_Receptacle_USB2.0_16P, J2 Conn_02x03_Pin, J3 Micro_SD_Card_Det1, J4 STARBOARD_SERVO, J5 PORTSIDE_SERVO, J6 Conn_01x02_Pin, J7 EJECTION_SERVO, Q1 BSS138, Q2 BSS138, Q3 BSS138, Q4 BSS138, U1 ATSAMD11D14A-M, U2 ATmega4809-A, U3 AT25DF641A-SH-T, U4 AP2112K-3.3, U5 BD1020HFV, U6 BNO086, U7 TXB0104D, U8 TPS61092, U9 MPM3610AGQV-P, Y1 32.768kHz

Commit message: not done 2.3 pcb
Parts:
- removed ?: , clipboard:b9f70def-b1a4-4804-8b04-89d3a63594a6
- removed REF** (x3): MountingHole_2.1mm, MountingHole:MountingHole_2.1mm
- added R8: DNP, Resistor_SMD:R_0402_1005Metric, F.Cu at (51.9, 57.9)
- moved U7 174.3 mm to (35.1, 189.3), turned to 180 degrees
- moved J3 157.5 mm to (45.7, 187.2)
- moved R21 155.1 mm to (27.6, 103.6)
- moved R22 154.4 mm to (27.6, 105.6)
- moved TP1 148.2 mm to (37.8, 20.2), turned to 90 degrees
- moved R23 147.5 mm to (50.1, 83.4), turned to -90 degrees
- moved D1 146.2 mm to (34.0, 19.6), turned to 90 degrees
- moved C2 145.0 mm to (43.8, 89.7), turned to 180 degrees
- moved R20 144.6 mm to (51.5, 85.6), turned to 0 degrees
- moved ADR1 144.4 mm to (52.2, 83.8), turned to 180 degrees
- moved C3 144.1 mm to (43.8, 90.6), turned to 180 degrees
- moved Y1 143.8 mm to (46.2, 89.1), turned to -90 degrees
- moved TP2 143.7 mm to (40.8, 20.2), turned to 90 degrees
- moved R19 142.7 mm to (53.0, 86.3), turned to 90 degrees
- moved U6 141.1 mm to (50.3, 89.0), turned to 90 degrees
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Routing:
- net +3.3V: track 175.7 -> 7.11 mm, vias 13 -> 0
- net GND: track 89.0 -> 24.4 mm, vias 44 -> 9
- net +5V: track 49.7 -> 8.48 mm
- net SCL: track 40.8 -> 0.00 mm, vias 2 -> 0
- net STAR_BLUE: track 37.2 -> 0.00 mm, vias 2 -> 0
- net STAR_GREEN: track 33.7 -> 0.00 mm, vias 4 -> 0
- net SDA: track 33.2 -> 0.00 mm
- net STAR_RED: track 33.1 -> 0.00 mm, vias 2 -> 0
- net D7: track 32.5 -> 0.00 mm, vias 2 -> 0
- net Net-(D1-GND): track 47.5 -> 15.2 mm, vias 4 -> 0
- net EJEC_SERVO: track 31.0 -> 0.00 mm, vias 2 -> 0
- net STAR_SERVO: track 30.0 -> 0.00 mm, vias 1 -> 0
- net TX0: track 29.5 -> 0.00 mm
- net D6: track 29.1 -> 0.00 mm, vias 2 -> 0
- net PA3/SS: track 28.7 -> 0.00 mm, vias 4 -> 0
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- added copper zone on B.Cu, net (none)
- added copper zone on F.Cu, net (none)
Other:
- board outline removed
- board text removed: "+ -"
- board text removed: "Portside"
- board text removed: "Starboard"

Commit message: transfer to v2.3
Parts:
- removed R8: DNP, Resistor_SMD:R_0402_1005Metric
- added ?: , clipboard:b9f70def-b1a4-4804-8b04-89d3a63594a6, F.Cu at (175.2, 112.2)
- added REF**: MountingHole_2.1mm, MountingHole:MountingHole_2.1mm, F.Cu at (154.8, 96.2)
- added REF**: MountingHole_2.1mm, MountingHole:MountingHole_2.1mm, F.Cu at (165.5, 132.0)
- added REF**: MountingHole_2.1mm, MountingHole:MountingHole_2.1mm, F.Cu at (181.0, 132.0)
- moved U7 174.3 mm to (185.8, 101.8), turned to -90 degrees
- moved J3 157.5 mm to (184.4, 112.7)
- moved R21 155.1 mm to (181.1, 126.0)
- moved R22 154.4 mm to (181.0, 123.8)
- moved TP1 148.2 mm to (156.7, 108.5), turned to 0 degrees
- moved R23 147.5 mm to (190.2, 129.3), turned to 90 degrees
- moved D1 146.2 mm to (154.7, 102.0), turned to 180 degrees
- moved C2 145.0 mm to (185.2, 121.5), turned to 90 degrees
- moved R20 144.6 mm to (189.3, 129.3), turned to -90 degrees
- moved ADR1 144.4 mm to (190.1, 126.7), turned to -90 degrees
- moved C3 144.1 mm to (184.5, 121.5), turned to 90 degrees
- moved Y1 143.8 mm to (185.7, 123.9), turned to 180 degrees
- moved TP2 143.7 mm to (154.2, 108.3), turned to 0 degrees
- moved R19 142.7 mm to (188.6, 130.7), turned to 0 degrees
- moved U6 141.1 mm to (185.8, 127.9), turned to 0 degrees
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Routing:
- net +3.3V: track 7.11 -> 175.7 mm, vias 0 -> 13
- net GND: track 24.4 -> 89.0 mm, vias 9 -> 44
- net +5V: track 8.48 -> 49.7 mm
- net SCL: track 0.00 -> 40.8 mm, vias 0 -> 2
- net STAR_BLUE: track 0.00 -> 37.2 mm, vias 0 -> 2
- net STAR_GREEN: track 0.00 -> 33.7 mm, vias 0 -> 4
- net SDA: track 0.00 -> 33.2 mm
- net STAR_RED: track 0.00 -> 33.1 mm, vias 0 -> 2
- net D7: track 0.00 -> 32.5 mm, vias 0 -> 2
- net Net-(D1-GND): track 15.2 -> 47.5 mm, vias 0 -> 4
- net EJEC_SERVO: track 0.00 -> 31.0 mm, vias 0 -> 2
- net STAR_SERVO: track 0.00 -> 30.0 mm, vias 0 -> 1
- net TX0: track 0.00 -> 29.5 mm
- net D6: track 0.00 -> 29.1 mm, vias 0 -> 2
- net PA3/SS: track 0.00 -> 28.7 mm, vias 0 -> 4
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- removed copper zone on B.Cu, net (none)
- removed copper zone on F.Cu, net (none)
Other:
- board outline added: 50 x 41.2 mm
- board text added: "+ -"
- board text added: "Portside"
- board text added: "Starboard"

Commit message: pcb
Parts:
- removed ?: , clipboard:b9f70def-b1a4-4804-8b04-89d3a63594a6
- removed REF** (x3): MountingHole_2.1mm, MountingHole:MountingHole_2.1mm
- added C11: 1u, Capacitor_SMD:C_0201_0603Metric, F.Cu at (259.7, 23.5)
- added R33: 5m, Resistor_SMD:R_0402_1005Metric, F.Cu at (265.8, 116.0)
- added R34: 2k2, Resistor_SMD:R_0402_1005Metric, F.Cu at (275.1, 69.7)
- added TP3: TestPoint, TestPoint:TestPoint_Pad_1.0x1.0mm, F.Cu at (58.0, 181.0)
- added TP4: TestPoint, TestPoint:TestPoint_Pad_1.0x1.0mm, F.Cu at (131.7, 162.7)
- added TP5: TestPoint, TestPoint:TestPoint_Pad_1.0x1.0mm, F.Cu at (115.8, 89.2)
- added TP6: TestPoint, TestPoint:TestPoint_Pad_1.0x1.0mm, F.Cu at (122.3, 88.5)
- added TP7: TestPoint, TestPoint:TestPoint_Pad_1.0x1.0mm, F.Cu at (127.7, 101.8)
- C2, C3: value 2p2 -> 22p
- C7: value 0u1F -> 0u1
- moved D5 156.5 mm to (266.0, 16.7), turned to 180 degrees
- moved C6 155.2 mm to (264.2, 17.5), turned to 0 degrees
- moved R17 154.8 mm to (264.4, 16.7)
- moved U4 152.5 mm to (264.8, 20.0), turned to 90 degrees
- moved R13 149.3 mm to (46.0, 20.0), turned to -45 degrees
- moved R16 147.8 mm to (263.5, 24.9), turned to -90 degrees
- moved R1 147.7 mm to (27.2, 33.2), turned to 90 degrees
- moved C5 147.5 mm to (262.7, 23.5), turned to -90 degrees
- moved R15 147.5 mm to (263.5, 23.0), turned to -90 degrees
- moved Q2 146.5 mm to (45.0, 22.5), turned to 45 degrees
- moved C1 146.2 mm to (28.1, 33.0), turned to 90 degrees
- moved R12 145.7 mm to (48.4, 22.4), turned to -45 degrees
- moved R10 145.5 mm to (43.1, 24.0), turned to -45 degrees
- moved Q1 145.5 mm to (39.6, 34.7), turned to -135 degrees
- moved U9 145.3 mm to (260.9, 20.6), turned to 0 degrees
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Connections:
- C1 pad 1: Net-(D1-GND) -> GND
- C4 pad 1: Net-(U9-IN) -> POWER_STAB
- C8 pad 1: Net-(D1-GND) -> POWER_STAB
- D1 pad 1: Net-(D1-GND) -> GND
- D1 pad 4: Net-(D1-GND) -> POWER_STAB
- D6 pad 2: Net-(D1-GND) -> POWER_STAB
- J1 pad A4: Net-(D1-GND) -> POWER_STAB
- J1 pad A9: Net-(D1-GND) -> POWER_STAB
- J1 pad B4: Net-(D1-GND) -> POWER_STAB
- J1 pad B9: Net-(D1-GND) -> POWER_STAB
- J6 pad 1: Net-(D1-GND) -> POWER_STAB
- L1 pad 1: Net-(D1-GND) -> Net-(L1-Pad1)
- Q4 pad 2: Net-(BZ1--) -> GND
- Q4 pad 3: GND -> Net-(BZ1--)
- R1 pad 1: Net-(D1-GND) -> GND
- R14 pad 1: Net-(U9-IN) -> POWER_STAB
- U2 pad 1: unconnected-(U2-PA5-Pad1) -> PA2/SCK
- U2 pad 2: unconnected-(U2-PA6-Pad2) -> PA1/MOSI
- U2 pad 3: TEMP_SENSOR -> PA0/MISO
- U2 pad 32: unconnected-(U2-PE2-Pad32) -> HOLD
- U2 pad 33: unconnected-(U2-PE3-Pad33) -> WP
- U2 pad 37: EJEC_SERVO -> SCL
- U2 pad 38: unconnected-(U2-PF4-Pad38) -> EJEC_SERVO
- U2 pad 4: SCL -> unconnected-(U2-PB0-Pad4)
- U2 pad 44: PA0/MISO -> unconnected-(U2-PA0-Pad44)
- U2 pad 45: PA1/MOSI -> unconnected-(U2-PA1-Pad45)
- U2 pad 46: PA2/SCK -> unconnected-(U2-PA2-Pad46)
- U2 pad 47: PA3/SS -> TEMP_SENSOR
- U2 pad 48: unconnected-(U2-PA4-Pad48) -> PA3/SS
- U3 pad 3: unconnected-(U3-~{WP}-Pad3) -> WP
- U3 pad 7: unconnected-(U3-~{HOLD}-Pad7) -> HOLD
- U8 pad 11: Net-(D1-GND) -> POWER_STAB
- U8 pad 8: Net-(D1-GND) -> POWER_STAB
- U9 pad 16: Net-(U9-IN) -> POWER_STAB
Routing:
- net +3.3V: track 175.7 -> 34.8 mm, vias 13 -> 0
- net Net-(D1-GND): track 47.5 -> 0.00 mm, vias 4 -> 0
- net +5V: track 49.7 -> 3.64 mm, vias 2 -> 0
- net SCL: track 40.8 -> 0.00 mm, vias 2 -> 0
- net STAR_BLUE: track 37.2 -> 0.00 mm, vias 2 -> 0
- net STAR_GREEN: track 33.7 -> 0.00 mm, vias 4 -> 0
- net SDA: track 33.2 -> 0.00 mm
- net STAR_RED: track 33.1 -> 0.00 mm, vias 2 -> 0
- net D7: track 32.5 -> 0.00 mm, vias 2 -> 0
- net EJEC_SERVO: track 31.0 -> 0.00 mm, vias 2 -> 0
- net STAR_SERVO: track 30.0 -> 0.00 mm, vias 1 -> 0
- net POWER_STAB: track 0.00 -> 29.8 mm, vias 0 -> 1
- net D6: track 29.1 -> 0.00 mm, vias 2 -> 0
- net PA3/SS: track 28.7 -> 0.00 mm, vias 4 -> 0
- net PA2/SCK: track 28.5 -> 0.00 mm, vias 4 -> 0
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- added copper zone on B.Cu, net (none)
- added copper zone on F.Cu, net (none)
Other:
- board size 50 x 41.2 mm -> 392.2 x 186.6 mm
- board text removed: "+ -"
- board text removed: "PCB Edge"
- board text removed: "Portside"
- board text removed: "Starboard"

Commit message: kicad
Parts:
- moved J6 180.2 mm to (95.0, 98.4), turned to 180 degrees
- moved C6 179.9 mm to (114.4, 117.1)
- moved R15 179.9 mm to (113.8, 122.6)
- moved C11 179.9 mm to (109.9, 123.1)
- moved C5 179.9 mm to (112.9, 123.0)
- moved D6 179.9 mm to (111.4, 124.8)
- moved R17 179.9 mm to (114.6, 116.3)
- moved U4 179.9 mm to (115.0, 119.6)
- moved U9 179.9 mm to (111.1, 120.2)
- moved C4 179.9 mm to (110.1, 116.6)
- moved D5 179.9 mm to (116.2, 116.2)
- moved R14 179.9 mm to (109.9, 117.5)
- moved R16 179.9 mm to (113.8, 124.5)
- moved C8 176.0 mm to (97.2, 97.6), turned to 90 degrees
- moved Q4 175.7 mm to (116.1, 133.6), turned to 180 degrees
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Routing:
- net +3.3V: track 34.8 -> 26.8 mm
- net SCL: track 0.00 -> 5.44 mm
- net Net-(PORTSIDE_RGB1-BA): track 0.00 -> 1.51 mm
- net Net-(STARBOARD_RGB1-BA): track 0.00 -> 1.50 mm
- net Net-(STARBOARD_RGB1-RA): track 0.00 -> 1.49 mm
- net Net-(STARBOARD_RGB1-GA): track 0.00 -> 1.49 mm
- net Net-(PORTSIDE_RGB1-RA): track 0.00 -> 1.49 mm
- net Net-(PORTSIDE_RGB1-GA): track 0.00 -> 1.49 mm
- net GND: track 87.4 -> 88.6 mm, vias 26 -> 28
- net Net-(J3-CLK): track 9.61 -> 8.61 mm
- net Net-(J3-DAT0): track 6.88 -> 6.04 mm
- net Net-(U6-XOUT32/CLKSEL1): track 5.98 -> 6.71 mm
- net Net-(J3-CMD): track 12.3 -> 11.8 mm
Other:
- board size 392.2 x 186.6 mm -> 42.1 x 52.7 mm

Commit message: pcb wiring
Parts:
- added REF**: MountingHole_2.1mm, MountingHole:MountingHole_2.1mm, F.Cu at (95.5, 87.0)
- added REF**: MountingHole_2.1mm, MountingHole:MountingHole_2.1mm, F.Cu at (131.5, 87.0)
- added REF**: MountingHole_2.1mm, MountingHole:MountingHole_2.1mm, F.Cu at (131.5, 133.0)
- moved BZ1 38.8 mm to (166.9, 119.5)
- moved R30 35.9 mm to (100.5, 108.5)
- moved PORTSIDE_RGB1 35.9 mm to (97.0, 109.5)
- moved R28 35.9 mm to (100.5, 110.5)
- moved R29 35.9 mm to (100.5, 109.5)
- moved R25 24.8 mm to (127.5, 109.0)
- moved R27 24.8 mm to (127.5, 111.0)
- moved R26 24.8 mm to (127.5, 110.0)
- moved STARBOARD_RGB1 24.8 mm to (131.0, 110.0)
- moved TP4 22.4 mm to (129.5, 121.5)
- moved U3 18.0 mm to (125.5, 121.5), turned to 90 degrees
- moved U5 15.2 mm to (118.5, 119.3), turned to 180 degrees
- moved J2 11.1 mm to (126.9, 106.0)
- moved J5 6.42 mm to (105.0, 86.4)
- moved J7 6.42 mm to (108.7, 86.4)
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Routing:
- net CD: track 0.00 -> 37.3 mm
- net D5: track 0.00 -> 34.0 mm, vias 0 -> 2
- net D6: track 0.00 -> 33.2 mm, vias 0 -> 2
- net D7: track 0.00 -> 32.3 mm
- net PORT_GREEN: track 0.00 -> 28.6 mm, vias 0 -> 2
- net PORT_RED: track 0.00 -> 27.0 mm, vias 0 -> 2
- net PORT_BLUE: track 0.00 -> 26.9 mm, vias 0 -> 2
- net +3.3V: track 26.8 -> 46.3 mm
- net WP: track 0.00 -> 19.2 mm
- net PA2/SCK: track 0.00 -> 13.4 mm
- net Net-(J2-Pin_6): track 13.0 -> 1.33 mm, vias 1 -> 0
- net PA0/MISO: track 0.00 -> 11.7 mm, vias 0 -> 2
- net Net-(J2-Pin_3): track 13.3 -> 2.09 mm, vias 1 -> 0
- net STAR_BLUE: track 0.00 -> 10.5 mm, vias 0 -> 2
- net Net-(J2-Pin_2): track 9.76 -> 0.00 mm, vias 2 -> 0
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
Commit message: layer fixes (kicad open)
Routing:
- net PORT_GREEN: track 28.6 -> 29.1 mm
Changed lines of the file:
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@@
 	)
 	(segment
-		(start 117.5 104)
-		(end 120 104)
-		(width 0.2)
-		(layer "In1.Cu")
+		(start 117 105.193588)
+		(end 117 106)
+		(width 0.2)
+		(layer "B.Cu")
 		(net 61)
 	)
 	(segment
-		(start 117 104.5)
-		(end 117.5 104)
-		(width 0.2)
-		(layer "In1.Cu")
+		(start 120 104)
+		(end 118.193588 104)
+		(width 0.2)
+		(layer "B.Cu")
 		(net 61)
 	)
 	(segment
-		(start 117 106)
-		(end 117 104.5)
-		(width 0.2)
-		(layer "In1.Cu")
+		(start 118.193588 104)
+		(end 117 105.193588)
+		(width 0.2)
+		(layer "B.Cu")
 		(net 61)
 	)
@@
 	)
 	(segment
-		(start 117.711062 105.331055)
+		(start 120.5 105)
 		(end 120.168945 105.331055)
 		(width 0.2)
-		(layer "In1.Cu")
+		(layer "B.Cu")
 		(net 63)
 	)
 	(segment
 		(start 120.168945 105.331055)
-		(end 120.5 105)
-		(width 0.2)
-		(layer "In1.Cu")
+		(end 117.711062 105.331055)
+		(width 0.2)
+		(layer "B.Cu")
 		(net 63)
 	)
@@
 	(segment
 		(start 123.5 121.805)
-		(end 123.5 117)
-		(width 0.2)
-		(layer "In1.Cu")
+		(end 124.195 122.5)
+		(width 0.2)
+		(layer "B.Cu")
 		(net 67)
 	)
 	(segment
-		(start 124.195 122.5)
+		(start 123.5 117)
 		(end 123.5 121.805)
 		(width 0.2)
-		(layer "In1.Cu")
+		(layer "B.Cu")
 		(net 67)
 	)
@@
 	)
 	(segment
-		(start 98.5 115.9)
+		(start 103.5 114.5)
 		(end 102.1 115.9)
 		(width 0.2)
-		(layer "In1.Cu")
+		(layer "B.Cu")
 		(net 70)
 	)
 	(segment
 		(start 102.1 115.9)
-		(end 103.5 114.5)
-		(width 0.2)
-		(layer "In1.Cu")
+		(end 98.5 115.9)
+		(width 0.2)
+		(layer "B.Cu")
 		(net 70)
 	)
@@
 	)
 	(segment
-		(start 112.95751 102.33757)
-		(end 112.95751 102.806039)
-		(width 0.2)
-		(layer "In1.Cu")
-		(net 105)
-	)
-	(segment
-		(start 115.5 108.5)
-		(end 117.861577 110.861577)
-		(width 0.2)
-		(layer "In1.Cu")
-		(net 105)
-	)
-	(segment
-		(start 117.861577 110.861577)
-		(end 117.861577 111.138423)
-		(width 0.2)
-		(layer "In1.Cu")
-		(net 105)
-	)
-	(segment
-		(start 112.95751 102.806039)
-		(end 115.5 105.348529)
-		(width 0.2)
-		(layer "In1.Cu")
-		(net 105)
-	)
-	(segment
-		(start 115.5 105.348529)
-		(end 115.5 108.5)
-		(width 0.2)
-		(layer "In1.Cu")
+		(start 117.6 111.4)
+		(end 117.6 110.1)
+		(width 0.2)
+		(layer "B.Cu")
+		(net 105)
+	)
+	(segment
+		(start 112.95751 102.95751)
+		(end 112.95751 102.33757)
+		(width 0.2)
+		(layer "B.Cu")
+		(net 105)
+	)
+	(segment
+		(start 117.6 110.1)
+		(end 115.5 108)
+		(width 0.2)
+		(layer "B.Cu")
+		(net 105)
+	)
+	(segment
+		(start 115.5 105.5)
+		(end 112.95751 102.95751)
+		(width 0.2)
+		(layer "B.Cu")
+		(net 105)
+	)
+	(segment
+		(start 115.5 108)
+		(end 115.5 105.5)
+		(width 0.2)
+		(layer "B.Cu")
+		(net 105)
+	)
+	(segment
+		(start 117.861577 111.138423)
+		(end 117.6 111.4)
+		(width 0.2)
+		(layer "B.Cu")
 		(net 105)
 	)
@@
 	)
 	(segment
+		(start 114.5 103)
+		(end 115.9 104.4)
+		(width 0.2)
+		(layer "B.Cu")
+		(net 107)
+	)
+	(segment
+		(start 115.9 104.4)
+		(end 115.9 105.9)
+		(width 0.2)
+		(layer "B.Cu")
+		(net 107)
+	)
+	(segment
 		(start 115.9 105.9)
 		(end 119 109)
 		(width 0.2)
-		(layer "In1.Cu")
-		(net 107)
-	)
-	(segment
-		(start 114.5 103)
-		(end 115.9 104.4)
-		(width 0.2)
-		(layer "In1.Cu")
-		(net 107)
-	)
-	(segment
-		(start 115.9 104.4)
-		(end 115.9 105.9)
-		(width 0.2)
-		(layer "In1.Cu")
+		(layer "B.Cu")
 		(net 107)
 	)
@@
 	)
 	(segment
+		(start 115 106)
+		(end 115 108.5)
+		(width 0.2)
+		(layer "B.Cu")
+		(net 108)
+	)
+	(segment
 		(start 112.5 103.5)
 		(end 115 106)
 		(width 0.2)
-		(layer "In1.Cu")
-		(net 108)
-	)
-	(segment
-		(start 115 107.5)
-		(end 115 109)
-		(width 0.2)
-		(layer "In1.Cu")
-		(net 108)
-	)
-	(segment
-		(start 115 106)
-		(end 115 107.5)
-		(width 0.2)
-		(layer "In1.Cu")
-		(net 108)
-	)
-	(segment
-		(start 115 109)
+		(layer "B.Cu")
+		(net 108)
+	)
+	(segment
+		(start 115 108.5)
+		(end 115.5 109)
+		(width 0.2)
+		(layer "B.Cu")
+		(net 108)
+	)
+	(segment
+		(start 115.5 109)
+		(end 115.5 109.5)
+		(width 0.2)
+		(layer "B.Cu")
+		(net 108)
+	)
+	(segment
+		(start 115.5 109.5)
 		(end 117 111)
 		(width 0.2)
-		(layer "In1.Cu")
-		(net 108)
-	)
+		(layer "B.Cu")
+		(net 108)
+	)

Commit message: not done wiring
Parts:
- moved BZ1 45.7 mm to (122.1, 128.9)
- moved R34 11.9 mm to (108.5, 128.9), turned to -90 degrees
- moved Q4 6.74 mm to (111.0, 129.2), turned to 0 degrees
- moved TP4 2.66 mm to (131.8, 120.1)
- moved U3 2.66 mm to (127.8, 120.1)
Routing:
- net +3.3V: track 46.3 -> 141.4 mm, vias 0 -> 14
- net +5V: track 6.50 -> 72.2 mm, vias 0 -> 2
- net EJEC_SERVO: track 0.00 -> 46.4 mm, vias 0 -> 1
- net POWER_STAB: track 39.5 -> 85.8 mm, vias 1 -> 5
- net UPDI: track 2.46 -> 47.0 mm, vias 0 -> 2
- net PORT_SERVO: track 0.00 -> 38.9 mm, vias 0 -> 1
- net STAR_SERVO: track 0.00 -> 32.5 mm, vias 0 -> 1
- net BUZZER: track 0.00 -> 28.6 mm, vias 0 -> 2
- net D4: track 9.44 -> 34.7 mm, vias 2 -> 6
- net SDA: track 0.00 -> 24.1 mm, vias 0 -> 4
- net Net-(J2-Pin_3): track 2.09 -> 22.6 mm, vias 0 -> 1
- net Net-(J2-Pin_6): track 1.33 -> 21.7 mm
- net Net-(J2-Pin_2): track 0.00 -> 18.9 mm, vias 0 -> 2
- net HOLD: track 0.00 -> 16.1 mm, vias 0 -> 2
- net GND: track 92.3 -> 104.7 mm, vias 34 -> 37
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